File: hardware/weigand.kicad_pcb (KiCad board)
At the start: 2 copper layers, 17.2 x 30.4 mm, 17 parts, among them K1 WIEGAND, P1 CONN_01X04, P2 CONN_01X04, Q1 FET_N, Q2 FET_N, U1 MDBT40, X1 32.768kHz

Commit message: updated hardwware
Connections:
- P2 pad 1: /GPIO_1 -> /TX_TTL
- P2 pad 2: /TX_TTL -> /DATA_0
- P2 pad 3: /RX_TTL -> /DATA_1
- U1 pad 26: /GPIO_1 -> Net-(U1-Pad26)
- U1 pad 29: /RX_TTL -> Net-(U1-Pad29)
Routing:
- net /DATA_0: track 12.5 -> 35.0 mm, vias 0 -> 1
- net /RX_TTL: track 19.7 -> 0.00 mm, vias 1 -> 0
- net /GPIO_1: track 9.93 -> 0.00 mm
- net /DATA_1: track 15.5 -> 24.4 mm, vias 0 -> 2
- net /TX_TTL: track 15.5 -> 12.8 mm
Other:
- board text added: "+"
- board text added: "BLEKey v1.2"
- board text removed: "BLEKey v1.0"
