File: hardware/weigand.sch (KiCad schematic (older format))
At the start: 17 parts, among them K1 WIEGAND, P1 CONN_01X04, P2 CONN_01X04, Q1 FET_N, Q2 FET_N, U1 MDBT40, X1 32.768kHz

Commit message: updated hardwware
Connections:
- net labels removed: GPIO_1, RX_TTL
- wire segments 62 -> 60
Changed lines of the file:
@@
 	1    0    0    -1
 $EndComp
-Text Label 9150 4150 0    60   ~ 0
+Text Label 8000 4150 0    60   ~ 0
 DATA_0
-Text Label 9150 4250 0    60   ~ 0
+Text Label 8000 4250 0    60   ~ 0
 DATA_1
 $Comp
@@
 Text Label 3450 3550 0    60   ~ 0
 TX_TTL
-Text Label 3450 3750 0    60   ~ 0
-RX_TTL
 Wire Wire Line
 	7550 1650 8800 1650
@@
 	10300 4150 10700 4150
 Wire Wire Line
-	9150 4150 9500 4150
-Wire Wire Line
-	9500 4250 9150 4250
-Wire Wire Line
 	7550 2000 8050 2000
 Wire Wire Line
@@
 	3400 3550 3850 3550
 Wire Wire Line
-	3400 3750 3850 3750
-Wire Wire Line
 	3400 4650 3850 4650
-Wire Wire Line
-	3400 3450 3850 3450
-Text Label 3450 3450 0    60   ~ 0
-GPIO_1
 Wire Wire Line
 	1900 2750 1700 2750
@@
 Wire Wire Line
 	8400 4350 8450 4350
+Text Label 8000 4050 0    60   ~ 0
+TX_TTL
 Wire Wire Line
 	8000 4050 8450 4050
-Text Label 8000 4050 0    60   ~ 0
-GPIO_1
-Text Label 8000 4150 0    60   ~ 0
-TX_TTL
-Text Label 8000 4250 0    60   ~ 0
-RX_TTL
+Wire Wire Line
+	9400 4450 9400 4350
+Wire Wire Line
+	9400 4350 9500 4350
+Text Label 9100 4150 0    60   ~ 0
+DATA_0
+Text Label 9100 4250 0    60   ~ 0
+DATA_1
 Wire Wire Line
 	8000 4150 8450 4150
 Wire Wire Line
-	8000 4250 8450 4250
-Wire Wire Line
-	9400 4450 9400 4350
-Wire Wire Line
-	9400 4350 9500 4350
+	8450 4250 8000 4250
+Wire Wire Line
+	9100 4150 9500 4150
+Wire Wire Line
+	9500 4250 9100 4250
 $EndSCHEMATC
